File: project/project.kicad_pcb (KiCad board)
At the start: 2 copper layers, 94.8 x 80.4 mm, 25 parts, among them SW1 SW_Push

Commit message: i did some update ig
Parts:
- removed SW1: SW_Push, Button_Switch_THT:SW_PUSH_6mm
- added SW2: SW_SPDT, footprint:SW-TH_SS-12F23-G040, F.Cu at (80.6, 37.7)
Routing:
- net +3V0: track 118.8 -> 87.5 mm
- net Net-(D1-A): track 202.8 -> 208.4 mm
